File: pcb/StickIt-Hat.sch (KiCad schematic (older format))
At the start: 33 parts, among them CON1 BARREL_JACK, J1 XuLA_IO_HDR, J3 JSHORTNORMAL, J4 JSHORTNORMAL, J5 JSHORTNORMAL, SW1 SW_PUSH, U1 NCV1117, U2 CAT24C32

Commit message: Added manufacturers part numbers to some of the parts.
Parts:
- C1, C3: manf# (none) -> UWX1C220MCL1GB
- C2, C4: manf# (none) -> LMK212BJ475KD-T
- C5: manf# (none) -> 08055C104KAT2A
- CON1: manf# (none) -> PJ-002A
- R1: manf# (none) -> RC0805JR-071KL
- RN1: manf# (none) -> 742C083392JP
- SW1: manf# (none) -> RS-282G05A3-SM RT
- U1: value NCV1117 -> AZ1117EH-3.3; manf# (none) -> AZ1117EH-3.3TRG1
- U2: manf# (none) -> CAT24C32WI-GT3
Changed lines of the file:
@@
 LIBS:memory
 LIBS:xilinx
-LIBS:special
 LIBS:microcontrollers
 LIBS:dsp
@@
 LIBS:xess
 LIBS:Cypress_PSoC
-LIBS:StickIt-RPi-cache
+LIBS:StickIt-Hat-cache
 EELAYER 25 0
 EELAYER END
@@
 F 2 "XESS:RS-282G05A3-SM_RT" H 3000 750 60  0001 C CNN
 F 3 "" H 3000 750 60  0000 C CNN
+F 4 "RS-282G05A3-SM RT" H 3000 750 60  0001 C CNN "manf#"
 	1    3000 750
 	1    0    0    -1
@@
 F 2 "Connect:BARREL_JACK" H 1100 7150 60  0001 C CNN
 F 3 "" H 1100 7150 60  0000 C CNN
+F 4 "PJ-002A" H 1100 7150 60  0001 C CNN "manf#"
 	1    1100 7150
 	1    0    0    -1
@@
 F 2 "Resistors_SMD:R_0805_HandSoldering" H 2738 7150 30  0001 C CNN
 F 3 "" H 2700 7300 60  0000 C CNN
+F 4 "LMK212BJ475KD-T" H 2700 7300 60  0001 C CNN "manf#"
 	1    2700 7300
 	1    0    0    -1
@@
 F 2 "Capacitors_SMD:c_elec_5x5.3" H 2350 7300 60  0001 C CNN
 F 3 "" H 2350 7300 60  0000 C CNN
+F 4 "UWX1C220MCL1GB" H 2350 7300 60  0001 C CNN "manf#"
 	1    2350 7300
 	1    0    0    -1
@@
 F 2 "Resistors_SMD:R_0805_HandSoldering" H 4188 7150 30  0001 C CNN
 F 3 "" H 4150 7300 60  0000 C CNN
+F 4 "LMK212BJ475KD-T" H 4150 7300 60  0001 C CNN "manf#"
 	1    4150 7300
 	1    0    0    -1
@@
 F 2 "Capacitors_SMD:c_elec_5x5.3" H 3800 7300 60  0001 C CNN
 F 3 "" H 3800 7300 60  0000 C CNN
+F 4 "UWX1C220MCL1GB" H 3800 7300 60  0001 C CNN "manf#"
 	1    3800 7300
 	1    0    0    -1
@@
 P 3400 6950
 F 0 "U1" H 3200 7050 50  0000 L BNN
-F 1 "NCV1117" H 3200 6975 50  0000 L BNN
+F 1 "AZ1117EH-3.3" H 3200 6975 50  0000 L BNN
 F 2 "XESS:SOT-223" H 3400 6900 50  0001 C CNN
 F 3 "" H 3400 6750 60  0000 C CNN
+F 4 "AZ1117EH-3.3TRG1" H 3400 6950 60  0001 C CNN "manf#"
 	1    3400 6950
 	1    0    0    -1
@@
 F 2 "SMD_Packages:SOIC-8-N" H 4500 4150 60  0001 C CNN
 F 3 "" H 4500 4150 60  0000 C CNN
+F 4 "CAT24C32WI-GT3" H 4500 4200 60  0001 C CNN "manf#"
 	1    4500 4200
 	1    0    0    -1
@@
 F 2 "XESS:CTS_742C043" H 5750 3750 50  0001 C CNN
 F 3 "" H 5750 3600 60  0000 C CNN
+F 4 "742C083392JP" H 5750 3600 60  0001 C CNN "manf#"
 	1    5750 3600
 	0    1    1    0
@@
 F 2 "Resistors_SMD:R_0805_HandSoldering" V 5230 3800 30  0001 C CNN
 F 3 "" H 5300 3800 30  0000 C CNN
+F 4 "RC0805JR-071KL" V 5300 3800 60  0001 C CNN "manf#"
 	1    5300 3800
 	1    0    0    -1
@@
 F 2 "Resistors_SMD:R_0805_HandSoldering" H 4788 3400 30  0001 C CNN
 F 3 "" H 4750 3550 60  0000 C CNN
+F 4 "08055C104KAT2A" H 4750 3550 60  0001 C CNN "manf#"
 	1    4750 3550
 	1    0    0    -1
@@
 1E 25 49 2A DA F6 C4 5C B7 0C C3 B9 A4 0A 98 09 FC 0D B0 92 CD 57 CD 1F 06 4E 04 26 A7 75 27 49
 52 39 26 13 73 DE C3 6C BE 70 B5 12 F8 16 86 73 8D C3 FF 03 63 F8 EE 2E BE 9A 04 B1 00 00 00 00
-49 45 4E 44 AE 42 60 82 72
+49 45 4E 44 AE 42 60 82 8E
 EndData
 $EndBitmap
